File: pcb/people-counter-74xx.sch (KiCad schematic (older format))
At the start: 46 parts

Commit message: Schema: improves - remove excessive AND2 gate, add SW to reset counter IC
Parts:
- removed U? (x4): 74LS08, symbol 74LS08
- added C1: 100n, symbol C
- added J1: Conn_01x02, symbol Conn_01x02
- added R2, R3: 10k, symbol R
- added RESET1: SW_Push, symbol SW_Push
- AFF1: renamed from AFF?; footprint (none) -> Displays_7-Segment:HDSP-78xx
- R7: renamed from R?; footprint (none) -> Resistors_SMD:R_0603_HandSoldering
- gave numbers to parts that had none: 39
- renumbered Detector_IN to Detector_IN1
Connections:
- net +5V: now also C1.2, RESET1.1
- net GND: now also U1.2 (R0(1)), U1.3 (R0(2)), U2.2 (R0(1)), U2.3 (R0(2)), U3.2 (R0(1)), U3.3 (R0(2)), U4.2 (R0(1)), U4.3 (R0(2)), R2.2, R3.1; no longer U1.6 (R9(1)), U1.7 (R9(2)), U4.6 (R9(1)), U4.7 (R9(2))
- net at U1.11 (Q3), U5.6 (D): now also U2.14 (CP0)
- net at U1.14 (CP0): now also J1.2 (Pin_2), R3.2; no longer R1.1
- net at U2.11 (Q3), U6.6 (D): now also U3.14 (CP0)
- net at U3.11 (Q3), U7.6 (D): now also U4.14 (CP0)
- net at U2.6 (R9(1)), U2.7 (R9(2)): now also U1.6 (R9(1)), U1.7 (R9(2)), U3.6 (R9(1)), U3.7 (R9(2)), U4.6 (R9(1)), U4.7 (R9(2)), C1.1, R2.1, RESET1.2
- new net: J1.1 (Pin_1), R1.1
Other:
- moved on the sheet: Detector_IN1, R1

Commit message: Schema: final version of schema
Parts:
- removed AFF1: HDSP-7xxx-A, Displays_7-Segment:HDSP-78xx, symbol HDSP-7xxx-A
- removed AFF2, AFF3, AFF4: HDSP-7xxx-A, symbol HDSP-7xxx-A
- added U10, U11, U12, U9: 7SEGMENT_CA, Displays_7-Segment:7SegmentLED_LTS6760_LTS6780, symbol 7SEGMENT_CA
- C1: footprint (none) -> Capacitors_SMD:C_0603_HandSoldering
- Detector_IN1: footprint (none) -> Pin_Headers:Pin_Header_Angled_1x03_Pitch2.54mm
- J2: renamed from J1; footprint (none) -> Pin_Headers:Pin_Header_Angled_1x02_Pitch2.54mm
- R1, R10, R11, R12, R13, R14, R15, R16, R17, R18, R19, R2, R20, R21, R22, R23, R24, R25, R26, R27, R28, R29, R3, R30, R31, R8, R9: footprint (none) -> Resistors_SMD:R_0603_HandSoldering
- R4: renamed from R5; footprint (none) -> Resistors_SMD:R_0603_HandSoldering
- R5: renamed from R6; footprint (none) -> Resistors_SMD:R_0603_HandSoldering
- R6: renamed from R4; footprint (none) -> Resistors_SMD:R_0603_HandSoldering
- U1: footprint (none) -> Housings_DIP:DIP-14_W7.62mm; OC_TME (none) -> SN74LS90D
- U2, U3, U4: footprint (none) -> Housings_DIP:DIP-14_W7.62mm
- U5, U6, U7, U8: footprint (none) -> Housings_DIP:DIP-16_W7.62mm; OC_GME (none) -> 421-032; OC_TME (none) -> SN74LS47D
Connections:
- net VCC is gone; now on net +5V: U1.5 (VCC), U2.5 (VCC), U3.5 (VCC), U4.5 (VCC), U5.16 (VCC), U6.16 (VCC), U7.16 (VCC), U8.16 (VCC)
- net +5V: now also U10.3 (CA), U10.5 (DP), U10.8 (CA), U11.3 (CA), U11.5 (DP), U11.8 (CA), U12.3 (CA), U12.5 (DP), U12.8 (CA), U9.3 (CA), U9.5 (DP), U9.8 (CA)
- net at R10.1: now also U9.10 (G)
- net at R4.1: now also U9.7 (A)
- net at R9.1: now also U9.9 (F)
- net at R8.1: now also U9.1 (E)
- net at R7.1: now also U9.2 (D)
- net at R6.1: now also U9.4 (C)
- net at R5.1: now also U9.6 (B)
- net at U6.11 (c): now also R13.2; no longer R11.2
- net at U6.12 (b): now also R12.2; no longer R13.2
- net at U6.13 (a): now also R11.2; no longer R12.2
- net at R17.1: now also U10.10 (G)
- net at R12.1: now also U10.6 (B)
- net at R16.1: now also U10.9 (F)
- net at R15.1: now also U10.1 (E)
- net at R14.1: now also U10.2 (D)
- net at R11.1: now also U10.7 (A)
- net at R13.1: now also U10.4 (C)
- net at U7.11 (c): now also R20.2; no longer R18.2
- net at U7.12 (b): now also R19.2; no longer R20.2
- net at U7.13 (a): now also R18.2; no longer R19.2
- net at R24.1: now also U11.10 (G)
- net at R19.1: now also U11.6 (B)
- net at R23.1: now also U11.9 (F)
- net at R22.1: now also U11.1 (E)
- net at R21.1: now also U11.2 (D)
- net at R18.1: now also U11.7 (A)
- net at R20.1: now also U11.4 (C)
- net at U8.11 (c): now also R27.2; no longer R25.2
- net at U8.12 (b): now also R26.2; no longer R27.2
- net at U8.13 (a): now also R25.2; no longer R26.2
- net at R31.1: now also U12.10 (G)
- net at R26.1: now also U12.6 (B)
- net at R30.1: now also U12.9 (F)
- net at R29.1: now also U12.1 (E)
- net at R28.1: now also U12.2 (D)
- net at R25.1: now also U12.7 (A)
- net at R27.1: now also U12.4 (C)
Other:
- moved on the sheet: C1, Detector_IN1, J2, R1, R10, R2, R3, R4, R5, R6, R7, R8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
